File: lockey.kicad_pcb (KiCad board)
At the start: 2 copper layers, 48.1 x 88.8 mm, 28 parts, among them J4 Conn_01x01, SW1 SW_PUSH, SW10 SW_PUSH, SW11 SW_PUSH, SW12 SW_PUSH, SW13 SW_PUSH, SW14 Rotary_Encoder, SW2 SW_PUSH, SW3 SW_PUSH, SW4 SW_PUSH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

Commit message: :sparkles: (all) create firstversion
Parts:
- L1, L2, L3, L4, L5: footprint swanmatch:YS-SK6812MINI-E -> mikamo3:YS-SK6812MINI-E_front; moved to F.Cu
Routing:
- net VCC: track 49.4 -> 89.9 mm
- net GND: track 224.5 -> 210.0 mm, vias 0 -> 5
- net Net-(L3-Pad2): track 20.6 -> 9.61 mm, vias 2 -> 0
- net Net-(L1-Pad2): track 20.6 -> 9.90 mm, vias 2 -> 0
- net Net-(L4-Pad2): track 20.3 -> 9.80 mm, vias 2 -> 0
- net Net-(L2-Pad2): track 20.3 -> 9.99 mm, vias 2 -> 0
- net LED: track 8.20 -> 14.1 mm, vias 1 -> 0
Other:
- outline, holes or cut-outs redrawn
- board text added: "WireLy v1.0 PCB designed by kamo"
