File: lockey.sch (KiCad schematic (older format))
At the start: 23 parts, among them SW1 SW_PUSH, SW10 SW_PUSH, SW11 SW_PUSH, SW12 SW_PUSH, SW13 SW_PUSH, SW14 Rotary_Encoder, SW2 SW_PUSH, SW3 SW_PUSH, SW4 SW_PUSH, SW5 SW_PUSH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

Commit message: :sparkles: (all) create firstversion
Parts:
- L1, L2, L3, L4, L5: footprint swanmatch:YS-SK6812MINI-E -> mikamo3:YS-SK6812MINI-E_front
Changed lines of the file:
@@
 F 0 "L1" H 1650 3962 51  0000 C CNN
 F 1 "SK6812MINI-E" H 1650 3897 16  0000 C CNN
-F 2 "swanmatch:YS-SK6812MINI-E" H 1650 3700 60  0001 C CNN
+F 2 "mikamo3:YS-SK6812MINI-E_front" H 1650 3700 60  0001 C CNN
 F 3 "" H 1650 3700 60  0001 C CNN
 	1    1650 3700
@@
 F 0 "L2" H 2250 3962 51  0000 C CNN
 F 1 "SK6812MINI-E" H 2250 3897 16  0000 C CNN
-F 2 "swanmatch:YS-SK6812MINI-E" H 2250 3700 60  0001 C CNN
+F 2 "mikamo3:YS-SK6812MINI-E_front" H 2250 3700 60  0001 C CNN
 F 3 "" H 2250 3700 60  0001 C CNN
 	1    2250 3700
@@
 F 0 "L3" H 2850 3962 51  0000 C CNN
 F 1 "SK6812MINI-E" H 2850 3897 16  0000 C CNN
-F 2 "swanmatch:YS-SK6812MINI-E" H 2850 3700 60  0001 C CNN
+F 2 "mikamo3:YS-SK6812MINI-E_front" H 2850 3700 60  0001 C CNN
 F 3 "" H 2850 3700 60  0001 C CNN
 	1    2850 3700
@@
 F 0 "L4" H 3450 3962 51  0000 C CNN
 F 1 "SK6812MINI-E" H 3450 3897 16  0000 C CNN
-F 2 "swanmatch:YS-SK6812MINI-E" H 3450 3700 60  0001 C CNN
+F 2 "mikamo3:YS-SK6812MINI-E_front" H 3450 3700 60  0001 C CNN
 F 3 "" H 3450 3700 60  0001 C CNN
 	1    3450 3700
@@
 F 0 "L5" H 4050 3962 51  0000 C CNN
 F 1 "SK6812MINI-E" H 4050 3897 16  0000 C CNN
-F 2 "swanmatch:YS-SK6812MINI-E" H 4050 3700 60  0001 C CNN
+F 2 "mikamo3:YS-SK6812MINI-E_front" H 4050 3700 60  0001 C CNN
 F 3 "" H 4050 3700 60  0001 C CNN
 	1    4050 3700
